File: LoROM 4Mbit/LoROM_4Mbit.kicad_pcb (KiCad board)
At the start: 2 copper layers, 101.1 x 36.1 mm, 7 parts, among them J1 Cartridge Connector, U1 PIC10F322, U2 SST39SF 010/020/040

Commit message: upload
Parts:
- removed G***: LOGO, yoey_footprints:ross_sit
Other:
- board text removed: "Art by Lockster"
